File: beam_kit_1.kicad_pcb (KiCad board)
At the start: 2 copper layers, 125 x 96 mm, 247 parts, among them J1 PZ2.54-2*20, J10 UART_SEPARATOR, J11 NRF, J12 BTN_KNOB, J13 BTN_KNOB, J14 KNOB_AND_WS, J15 dbg, J16 dbg, J17 dbg, J18 dbg, J19 SONAR, J2 PZ2.54-2*20, J20 micro_sd, J21 NRF_24_socket, J22 SSD1306_128x32_OLED, J23 3V3, J24 GND, J25 5V, J27 PJ-320D, J28 screw_term, J29 screw_term, J3 USB_C_Receptacle, J30 RS485, J32 AUDIO, J4 probe_debug, J5 Micro_SD_Card, J6 OLED I2C, J7 VL53_PINS, J8 HC-SR04, J9 I2C, SW1 BOOTSEL, SW2 RUN, SW4 BTN1, SW5 BTN0, SW6 BTN2, SW7 RUN, U1 LIS3DH, U10 SHT30-DIS, U11 AMS1117-3.3, U12 SN74LVC1G14DBV, U13 SN74LVC1G14DBV, U14 MAX485E, U16 LMV358IDR, U2 APDS-9306-065, U3 SN74LVC1G14DBV, U4 M24256-BR, U5 RP2040, U6 SN74LVC1G14DBV, U7 W25Q16JVSS, U8 MT3608, U9 VL53L0CXV0DH1, Y1 12 MHz

Commit message: kju fix and PCB size increase
Parts:
- removed R42: 120R 1%, Resistor_SMD:R_0603_1608Metric_Pad0.98x0.95mm_HandSolder
- added J26: EXP-A, Connector_PinHeader_2.54mm:PinHeader_1x06_P2.54mm_Vertical, F.Cu at (78.5, 173.7)
- added J31: ~, Connector_PinSocket_2.54mm:PinSocket_1x06_P2.54mm_Vertical, F.Cu at (78.5, 178.3)
- moved JP5 223.0 mm to (253.6, 62.8), turned to 180 degrees
- moved C1 219.7 mm to (242.5, 65.7)
- moved U1 219.7 mm to (250.2, 62.8)
- moved C2 219.7 mm to (245.0, 65.7)
- moved C3 219.7 mm to (247.5, 65.7)
- moved U2 219.7 mm to (249.6, 58.1)
- moved U4 219.7 mm to (244.6, 59.4)
- moved U10 217.0 mm to (252.2, 68.0)
- moved C53 209.9 mm to (247.7, 71.6)
- moved C54 209.9 mm to (247.7, 74.1)
- moved C55 209.9 mm to (247.7, 76.6)
- moved C56 209.9 mm to (247.7, 79.2)
- moved C57 209.9 mm to (247.7, 81.7)
- moved R23 209.9 mm to (243.5, 76.6)
- moved R24 209.9 mm to (243.5, 79.2)
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Connections:
- R45 pad 2: Net-(D39-TVS2) -> Net-(D39-TVS3)
Other:
- board size 125 x 96 mm -> 145 x 96 mm
- board text added: "+"
- board text added: "-"
- board text added: "DEBUG UART CONNECT"

Commit message: layout
Parts:
- added D40: LED R, LED_SMD:LED_0603_1608Metric_Pad1.05x0.95mm_HandSolder, F.Cu at (121.7, 53.9)
- added D41: LED R, LED_SMD:LED_0603_1608Metric_Pad1.05x0.95mm_HandSolder, F.Cu at (110.5, 53.9)
- added H8: Hole, MountingHole:MountingHole_3.2mm_M3_Pad_Via, F.Cu at (153.5, 62.0)
- added R42: 10k 1%, Resistor_SMD:R_0603_1608Metric_Pad0.98x0.95mm_HandSolder, F.Cu at (119.3, 55.5)
- added R54: 10k 1%, Resistor_SMD:R_0603_1608Metric_Pad0.98x0.95mm_HandSolder, F.Cu at (112.9, 55.5)
- added kibuzzard-67BB2A29: G***, kibuzzard-67BB2A29, F.Cu at (117.7, 113.4)
- added kibuzzard-67BB2A6B: G***, kibuzzard-67BB2A6B, F.Cu at (160.0, 110.8)
- added kibuzzard-67BB2BB0: G***, kibuzzard-67BB2BB0, F.Cu at (92.8, 98.9)
- added kibuzzard-67BB2C58: G***, kibuzzard-67BB2C58, F.Cu at (91.6, 117.7)
- added kibuzzard-67BB2CB4: G***, kibuzzard-67BB2CB4, F.Cu at (208.8, 62.6)
- added kibuzzard-67BB2CE4: G***, kibuzzard-67BB2CE4, F.Cu at (169.3, 115.1)
- added kibuzzard-67BB2D55: G***, kibuzzard-67BB2D55, F.Cu at (190.6, 128.4)
- added kibuzzard-67BB2D66: G***, kibuzzard-67BB2D66, F.Cu at (168.4, 128.4)
- added kibuzzard-67BB2DE0: G***, kibuzzard-67BB2DE0, F.Cu at (92.4, 60.1)
- added kibuzzard-67BB2E05: G***, kibuzzard-67BB2E05, F.Cu at (201.3, 145.3)
- added kibuzzard-67BB2F8C: G***, kibuzzard-67BB2F8C, F.Cu at (187.2, 109.0)
- added kibuzzard-67BB2FFD: G***, kibuzzard-67BB2FFD, F.Cu at (116.1, 53.5)
- moved J32 106.3 mm to (157.2, 118.9), turned to 180 degrees
- moved J25 96.1 mm to (120.9, 73.0), turned to 180 degrees
- moved J24 94.8 mm to (117.2, 73.0), turned to 180 degrees
- moved J23 93.9 mm to (111.0, 73.0), turned to 180 degrees
- moved SW7 65.0 mm to (194.6, 109.1), turned to 90 degrees
- moved R12 64.6 mm to (197.1, 109.2)
- moved D37 60.0 mm to (132.2, 131.0)
- moved R43 58.2 mm to (114.4, 116.7), turned to -90 degrees
- moved C64 57.9 mm to (120.2, 122.5)
- moved C72 57.7 mm to (124.1, 114.4), turned to 0 degrees
- moved D36 56.2 mm to (116.8, 131.0), turned to 180 degrees
- moved R44 56.1 mm to (117.4, 116.7), turned to -90 degrees
- moved U14 55.7 mm to (116.4, 122.5)
- moved D39 54.5 mm to (124.2, 117.4), turned to -90 degrees
- moved R45 54.2 mm to (120.4, 116.7), turned to -90 degrees
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Connections:
- D38 pad 1: Net-(D38-TVS1) -> /peripheral2/CH_RIGHT
- D38 pad 3: /peripheral2/CH_RIGHT -> Net-(D38-TVS2)
- D5 pad 1: +3.3V -> unconnected-(D5-TVS1-Pad1)
- J2 pad 10: +3.3V -> unconnected-(D5-TVS1-Pad1)
- J2 pad 9: +3.3V -> unconnected-(D5-TVS1-Pad1)
- J32 pad 3: Net-(D38-TVS1) -> Net-(D38-TVS2)
- R53 pad 1: Net-(D38-TVS1) -> Net-(D38-TVS2)
Routing:
- net +3.3V: track 37.9 -> 24.7 mm
- net unconnected-(D5-TVS1-Pad1): track 0.00 -> 7.05 mm
Other:
- board text added: "0"
- board text added: "1"
- board text added: "10"
- board text added: "11"
- board text added: "12"
- board text added: "13"
- board text added: "14"
- board text added: "15"
- board text added: "16"
- board text added: "17"
- board text added: "18"
- board text added: "19"
- board text added: "2"
- board text added: "20"
- board text added: "21"
- board text added: "22"
- board text added: "26"
- board text added: "27"
- board text added: "28"
- board text added: "3"
- board text added: "3V3"
- board text added: "4"
- board text added: "5"
- board text added: "6"
- board text added: "7"
- board text added: "8"
- board text added: "9"
- board text added: "A"
- board text added: "B"
- board text added: "DE ~{RE}"
- board text added: "DI"
- board text added: "HC-SR04 SOCKET"
- board text added: "KNOB"
- board text added: "MIC"
- board text added: "MIC VOL"
- board text added: "OUT_L"
- board text added: "OUT_R"
- board text added: "RO"
- board text removed: "3V3 PICO"
- board text removed: "GPIO10"
- board text removed: "GPIO11"
- board text removed: "GPIO12"
- board text removed: "GPIO13"
- board text removed: "GPIO14"
- board text removed: "GPIO15"
- board text removed: "GPIO16"
- board text removed: "GPIO17"
- board text removed: "GPIO18"
- board text removed: "GPIO19"
- board text removed: "GPIO2"
- board text removed: "GPIO20"
- board text removed: "GPIO21"
- board text removed: "GPIO22"
- board text removed: "GPIO26"
- board text removed: "GPIO27"
- board text removed: "GPIO28"
- board text removed: "GPIO3"
- board text removed: "GPIO4"
- board text removed: "GPIO5"
- board text removed: "GPIO6"
- board text removed: "GPIO7"
- board text removed: "GPIO8"
- board text removed: "GPIO9"
- board text removed: "HC-SR04 SONAR SOCKET"
- board text removed: "NRF24 SOCKET"
- board text removed: "OLED"
- board text removed: "POT"
- board text removed: "USER BUTTONS"
- board text removed: "USER LEDs"
- board text removed: "microSD"

Commit message: layout
Parts:
- added kibuzzard-67BB32E4: G***, kibuzzard-67BB32E4, F.Cu at (117.2, 61.2)
- moved D34 138.8 mm to (120.0, 71.6)
- moved U11 135.3 mm to (121.0, 77.5), turned to -90 degrees
- moved C59 134.3 mm to (119.2, 67.1), turned to 90 degrees
- moved C58 129.4 mm to (122.5, 67.1), turned to 90 degrees
- moved J31 128.5 mm to (110.9, 54.0), turned to 90 degrees
- moved J26 119.5 mm to (110.9, 58.6), turned to 90 degrees
- moved D40 12.5 mm to (115.0, 64.5)
- moved D41 12.5 mm to (103.8, 64.5)
- moved J23 12.5 mm to (104.3, 83.5)
- moved J24 12.5 mm to (110.5, 83.5)
- moved J25 12.5 mm to (114.2, 83.5)
- moved R42 12.5 mm to (112.6, 66.1)
- moved R54 12.5 mm to (106.2, 66.1)
- moved kibuzzard-67BB2FFD 12.4 mm to (109.4, 63.9)
Connections:
- A1 pad 35: unconnected-(A1-ADC_VREF-Pad35)_1 -> /VREF
- A2 pad 35: unconnected-(A2-ADC_VREF-Pad35) -> /VREF
- D5 pad 3: unconnected-(D5-TVS2-Pad3) -> /VREF
- J2 pad 11: unconnected-(D5-TVS2-Pad3) -> /VREF
- J2 pad 12: unconnected-(D5-TVS2-Pad3) -> /VREF
Routing:
- net unconnected-(D5-TVS2-Pad3): track 8.42 -> 0.00 mm
- net /VREF: track 0.00 -> 8.42 mm
Other:
- board text added: "DEBUG UART"
- board text added: "VREF"
- board text removed: "DEBUG UART CONNECT"
