File: beam_kit_1.kicad_pcb (KiCad board)
At the start: 2 copper layers, 145 x 96 mm, 276 parts, among them J1 PZ2.54-2*20, J10 UART_SEPARATOR, J11 NRF, J12 BTN_KNOB, J13 BTN_KNOB, J14 KNOB_AND_WS, J15 dbg, J16 dbg, J17 dbg, J18 dbg, J19 SONAR, J2 PZ2.54-2*20, J20 micro_sd, J21 NRF_24_socket, J22 SSD1306_128x32_OLED, J23 3V3, J24 GND, J25 5V, J26 TERM, J27 PJ-320D, J28 screw_term, J29 screw_term, J3 USB_C_Receptacle, J30 RS485, J32 AUDIO, J33 EXP, J34 EXP, J4 probe_debug, J5 Micro_SD_Card, J6 OLED I2C, J7 VL53_PINS, J8 HC-SR04, J9 I2C, SW1 BOOTSEL, SW2 RUN, SW4 BTN1, SW5 BTN0, SW6 BTN2, SW7 RUN, U1 LIS3DH, U10 SHT30-DIS, U11 AMS1117-3.3, U12 SN74LVC1G14DBV, U13 SN74LVC1G14DBV, U14 MAX485E, U16 LMV358IDR, U2 APDS-9306-065, U3 SN74LVC1G14DBV, U4 M24256-BR, U5 RP2040, U6 SN74LVC1G14DBV, U7 W25Q16JVSS, U8 MT3608, U9 VL53L0CXV0DH1, Y1 12 MHz

Commit message: corrections
Parts:
- removed C1: 1u 50V, Capacitor_SMD:C_0603_1608Metric_Pad1.08x0.95mm_HandSolder
- removed U2: APDS-9306-065, OptoDevice:Broadcom_DFN-6_2x2mm_P0.65mm
- moved C55 5.16 mm to (110.9, 96.1)
- moved U10 5.16 mm to (108.3, 96.1)
Routing:
- net GND: track 1677.6 -> 1668.0 mm, vias 626 -> 671
- net +3.3V: track 698.1 -> 692.3 mm
- net /peripheral/SCL: track 52.0 -> 49.3 mm, vias 7 -> 5
- net /peripheral/SDA: track 48.7 -> 48.0 mm, vias 5 -> 4
Other:
- board text added: "BOOT"
- board text added: "G"
- board text added: "SWD"
- board text added: "TGrx"
- board text added: "TGtx"
- board text removed: "LIGHT SENSOR"

Commit message: final version
Parts:
- moved R47 14.8 mm to (138.8, 146.2), turned to -90 degrees
- moved R46 3.72 mm to (139.0, 138.4)
- moved J29 0.70 mm to (128.9, 139.8)
- moved MK1 0.45 mm to (142.9, 140.5)
- moved J28 0.20 mm to (116.1, 139.8)
Routing:
- net Net-(U16A-+): track 12.3 -> 23.7 mm
- net GND: track 1668.0 -> 1673.7 mm, vias 671 -> 668
- net /peripheral2/A: track 38.6 -> 40.4 mm
- net +3.3V: track 692.3 -> 693.3 mm
- net /peripheral2/B: track 46.7 -> 47.2 mm
