File: peripheral.kicad_sch (KiCad schematic)
At the start: 49 parts, among them J11 NRF, J19 SONAR, J20 micro_sd, J21 NRF_24_socket, J22 SSD1306_128x32_OLED, J33 EXP, J34 EXP, J5 Micro_SD_Card, J6 OLED I2C, J7 VL53_PINS, J8 HC-SR04, J9 I2C, U1 LIS3DH, U10 SHT30-DIS, U2 APDS-9306-065, U4 M24256-BR, U6 SN74LVC1G14DBV, U8 MT3608, U9 VL53L0CXV0DH1

Commit message: layout done
Connections:
- net +3V3 renamed +3.3V

Commit message: corrections
Parts:
- removed C1: 1u 50V, Capacitor_SMD:C_0603_1608Metric_Pad1.08x0.95mm_HandSolder, symbol Device:C_Small
- removed U2: APDS-9306-065, OptoDevice:Broadcom_DFN-6_2x2mm_P0.65mm, symbol Sensor_Optical:APDS-9306-065
Connections:
- no-connect marks 8 -> 7
Other:
- note removed: "Sensor address: 0x52 (0b1010010)"

Commit message: final version
Parts:
- C19, C2, C31, C34, C35, C54, C56: JLC (none) -> C19702
- C3, C32, C53, C55, C57: JLC (none) -> C14663
- D14: JLC (none) -> C2960361
- J11, J20: JLC (none) -> C37208
- J19: JLC (none) -> C49257
- J21: JLC (none) -> C92271
- J22, J8: JLC (none) -> C2718488
- J33: JLC (none) -> C18078205
- J34: JLC (none) -> C5224027
- J5: JLC (none) -> C585350
- J6, J7, J9: JLC (none) -> C492401
- L1: JLC (none) -> C139250
- R11, R17, R23, R24, R36, R9: JLC (none) -> C25804
- R16: JLC (none) -> C23186
- R18: JLC (none) -> C25805
- R19: JLC (none) -> C22809
- R21, R22, R25, R26: JLC (none) -> C4190
- U1: JLC (none) -> C15134
- U10: JLC (none) -> C2687423
- U4: JLC (none) -> C79984
- U6: JLC (none) -> C7835
- U8: JLC (none) -> C84817
- U9: JLC (none) -> C91199
