File: beam_kit_1.kicad_sch (KiCad schematic)
At the start: 43 parts, among them J1 PZ2.54-2*20, J10 UART_SEPARATOR, J15 dbg, J16 dbg, J17 dbg, J18 dbg, J2 PZ2.54-2*20, SW7 RUN, U11 AMS1117-3.3

Commit message: codes and fixes
Parts:
- C21, C22, C23, C24, C25, C26, C27, C28, C29, C30: jlc (none) -> C14663
- D34: value 1A, 30V -> 2A, 30V; MPN DFLS130-7 -> DFLS230LH-7; jlc C150474 -> C2960361
- J10: jlc (none) -> C7501273
- J15, J16, J17, J18: jlc (none) -> C495538; now fitted
Changed lines of the file:
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@@
 		(in_bom yes)
 		(on_board yes)
-		(dnp yes)
+		(dnp no)
 		(property "Reference" "J17"
 			(at 136.652 166.116 0)
@@
 			)
 		)
+		(property "jlc" "C495538"
+			(at 138.43 161.29 0)
+			(effects
+				(font
+					(size 1.27 1.27)
+				)
+				(hide yes)
+			)
+		)
 		(pin "1"
 		)
@@
 			)
 		)
+		(property "jlc" "C14663"
+			(at 224.79 82.55 0)
+			(effects
+				(font
+					(size 1.27 1.27)
+				)
+				(hide yes)
+			)
+		)
 		(pin "1"
 		)
@@
 			)
 		)
+		(property "jlc" "C14663"
+			(at 224.79 100.33 0)
+			(effects
+				(font
+					(size 1.27 1.27)
+				)
+				(hide yes)
+			)
+		)
 		(pin "1"
 		)
@@
 			)
 		)
+		(property "jlc" "C14663"
+			(at 224.79 110.49 0)
+			(effects
+				(font
+					(size 1.27 1.27)
+				)
+				(hide yes)
+			)
+		)
 		(pin "1"
 		)
@@
 		(in_bom yes)
 		(on_board yes)
-		(dnp yes)
+		(dnp no)
 		(property "Reference" "J15"
 			(at 125.222 156.464 0)
@@
 			)
 		)
+		(property "jlc" "C495538"
+			(at 127 161.29 0)
+			(effects
+				(font
+					(size 1.27 1.27)
+				)
+				(hide yes)
+			)
+		)
 		(pin "1"
 		)
@@
 			)
 		)
+		(property "jlc" "C14663"
+			(at 224.79 62.23 0)
+			(effects
+				(font
+					(size 1.27 1.27)
+				)
+				(hide yes)
+			)
+		)
 		(pin "1"
 		)
@@
 			)
 		)
+		(property "jlc" "C14663"
+			(at 224.79 72.39 0)
+			(effects
+				(font
+					(size 1.27 1.27)
+				)
+				(hide yes)
+			)
+		)
 		(pin "1"
 		)
@@
 			)
 		)
+		(property "jlc" "C14663"
+			(at 224.79 130.81 0)
+			(effects
+				(font
+					(size 1.27 1.27)
+				)
+				(hide yes)
+			)
+		)
 		(pin "1"
 		)
@@
 			)
 		)
+		(property "jlc" "C14663"
+			(at 224.79 41.91 0)
+			(effects
+				(font
+					(size 1.27 1.27)
+				)
+				(hide yes)
+			)
+		)
 		(pin "1"
 		)
@@
 			)
 		)
-		(property "Value" "1A, 30V"
+		(property "Value" "2A, 30V"
 			(at 171.704 24.13 0)
 			(effects
@@
 			)
 		)
-		(property "MPN" "DFLS130-7"
+		(property "MPN" "DFLS230LH-7"
 			(at 171.45 21.59 0)
 			(effects
@@
 			)
 		)
-		(property "jlc" "C150474"
+		(property "jlc" "C2960361"
 			(at 171.45 21.59 0)
 			(effects
@@
 			)
 		)
+		(property "jlc" "C7501273"
+			(at 153.67 175.26 0)
+			(effects
+				(font
+					(size 1.27 1.27)
+				)
+				(hide yes)
+			)
+		)
 		(pin "4"
 		)
@@
 			)
 		)
+		(property "jlc" "C14663"
+			(at 224.79 52.07 0)
+			(effects
+				(font
+					(size 1.27 1.27)
+				)
+				(hide yes)
+			)
+		)
 		(pin "1"
 		)
@@
 			)
 		)
+		(property "jlc" "C14663"
+			(at 224.79 120.65 0)
+			(effects
+				(font
+					(size 1.27 1.27)
+				)
+				(hide yes)
+			)
+		)
 		(pin "1"
 		)
@@
 			)
 		)
+		(property "jlc" "C14663"
+			(at 224.79 140.97 0)
+			(effects
+				(font
+					(size 1.27 1.27)
+				)
+				(hide yes)
+			)
+		)
 		(pin "1"
 		)
@@
 		(in_bom yes)
 		(on_board yes)
-		(dnp yes)
+		(dnp no)
 		(property "Reference" "J18"
 			(at 136.652 178.816 0)
@@
 			)
 		)
+		(property "jlc" "C495538"
+			(at 138.43 173.99 0)
+			(effects
+				(font
+					(size 1.27 1.27)
+				)
+				(hide yes)
+			)
+		)
 		(pin "1"
 		)
@@
 		(in_bom yes)
 		(on_board yes)
-		(dnp yes)
+		(dnp no)
 		(property "Reference" "J16"
 			(at 125.222 169.164 0)
@@
 			(at 127 173.99 0)
 			(effects
+				(font
+					(size 1.27 1.27)
+				)
+				(hide yes)
+			)
+		)
+		(property "jlc" "C495538"
+			(at 127 173.99 0)
+			(effects

Commit message: jlc codes filled
Parts:
- R12: jlc (none) -> C25804
Changed lines of the file:
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@@
+			)
+		)
+		(property "jlc" "C25804"
+			(at 116.84 118.11 0)
+			(effects
+				(font
+					(size 1.27 1.27)
+				)
+				(hide yes)
 			)
 		)

Commit message: routing in progress
Parts:
- R12: now left out of the parts list
Changed lines of the file:
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@@
 		(unit 1)
 		(exclude_from_sim no)
-		(in_bom yes)
+		(in_bom no)
 		(on_board yes)
 		(dnp yes)

Commit message: layout done
Connections:
- net RUN: now also A1.30 (RUN), R12.1, SW7.2
Changed lines of the file:
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@@
+		)
+	)
+	(label "RUN"
+		(at 116.84 109.22 0)
+		(fields_autoplaced yes)
+		(effects
+			(font
+				(size 1.27 1.27)
+			)
+			(justify left bottom)
 		)
 	)

Commit message: final version
Parts:
- A2: now left out of the parts list
- C21, C22, C23, C24, C25, C26, C27, C28, C29, C30: JLC (none) -> C14663
- C58, C59: JLC (none) -> C16133
- D10, D11, D12, D13, D4, D5, D6, D7, D8, D9: JLC (none) -> C495220
- D34: JLC (none) -> C2960361
- J1, J2: JLC (none) -> C5224014
- J10: JLC (none) -> C7501273
- J15, J16, J17, J18: JLC (none) -> C495538
- R12: JLC (none) -> C25804
- SW7: JLC (none) -> C231329
- U11: JLC (none) -> C6186
