File: buttons_LEDs.kicad_sch (KiCad schematic)
At the start: 49 parts, among them J12 BTN_KNOB, J13 BTN_KNOB, J14 KNOB_AND_WS, SW4 BTN1, SW5 BTN0, SW6 BTN2, U3 SN74LVC1G14DBV

Commit message: final version
Parts:
- C33, C36, C37, C38, C39, C40, C43, C44, C45, C46, C47, C48, C49, C50, C51, C52: JLC (none) -> C1525
- C41, C42: JLC (none) -> C14663
- D15, D16, D17: JLC (none) -> C2286
- D18, D19, D20, D21, D22, D23, D24, D25, D26, D27, D28, D29, D30, D31, D32, D33: JLC (none) -> C2843785
- J12, J13: JLC (none) -> C49257
- J14: JLC (none) -> C492401
- R14, R15, R20: JLC (none) -> C23186
- R38: JLC (none) -> C25804
- RV2: JLC (none) -> C116302
- SW4, SW5, SW6: JLC (none) -> C455112
- U3: JLC (none) -> C7835
