File: prog.kicad_sch (KiCad schematic)
At the start: 39 parts, among them J3 USB_C_Receptacle, J4 probe_debug, SW1 BOOTSEL, SW2 BOOTSEL, U5 RP2040, U7 W25Q16JVSS, Y1 12 MHz

Commit message: fit test
Parts:
- added R27, R28, R29, R30: 100R 1%, Resistor_SMD:R_0603_1608Metric_Pad0.98x0.95mm_HandSolder, symbol Device:R_Small
- SW1: footprint Button_Switch_SMD:SW_Push_1P1T_NO_6x6mm_H9.5mm -> Button_Switch_SMD:SW_SPST_B3U-1000P; jlc (none) -> C231329
- SW2: value BOOTSEL -> RUN; footprint Button_Switch_SMD:SW_Push_1P1T_NO_6x6mm_H9.5mm -> Button_Switch_SMD:SW_SPST_B3U-1000P; jlc (none) -> C231329
Connections:
- net TARGET_RX: now also R28.1; no longer JP2.2 (B), JP3.2 (B)
- net TARGET_SWCLK: now also R29.1; no longer U5.4 (GPIO2)
- net TARGET_SWDIO: now also R30.1; no longer U5.5 (GPIO3)
- net TARGET_TX: now also R27.1; no longer JP1.2 (B), JP4.2 (B)
- new net: JP2.2 (B), JP3.2 (B), R28.2
- new net: R30.2, U5.5 (GPIO3)
- new net: R29.2, U5.4 (GPIO2)
- new net: JP1.2 (B), JP4.2 (B), R27.2
- no-connect marks 10 -> 35

Commit message: more stuff added to sch
Parts:
- JP1, JP2, JP3, JP4: now left out of the parts list
Changed lines of the file:
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@@
 		(unit 1)
 		(exclude_from_sim yes)
-		(in_bom yes)
+		(in_bom no)
 		(on_board yes)
 		(dnp no)
@@
 		(unit 1)
 		(exclude_from_sim yes)
-		(in_bom yes)
+		(in_bom no)
 		(on_board yes)
 		(dnp no)
@@
 		(unit 1)
 		(exclude_from_sim yes)
-		(in_bom yes)
+		(in_bom no)
 		(on_board yes)
 		(dnp no)
@@
 		(unit 1)
 		(exclude_from_sim yes)
-		(in_bom yes)
-		(on_board yes)
-		(dnp no)
+		(in_bom no)
+		(on_board yes)
+		(dnp no)

Commit message: codes and fixes
Parts:
- C10, C11, C12, C13, C15, C16, C20, C4, C6, C7, C8, C9: jlc (none) -> C14663
- C14, C5: jlc (none) -> C15849
- D2: value 1A, 30V -> 2A, 30V; MPN DFLS130-7 -> DFLS230LH-7; jlc C150474 -> C2960361
- D3: jlc (none) -> C2286
- J4: jlc (none) -> C49257
Changed lines of the file:
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@@
 			)
 		)
+		(property "jlc" "C14663"
+			(at 153.67 33.02 0)
+			(effects
+				(font
+					(size 1.27 1.27)
+				)
+				(hide yes)
+			)
+		)
 		(pin "1"
 		)
@@
 			)
 		)
+		(property "jlc" "C14663"
+			(at 213.36 40.64 0)
+			(effects
+				(font
+					(size 1.27 1.27)
+				)
+				(hide yes)
+			)
+		)
 		(pin "1"
 		)
@@
 			)
 		)
+		(property "jlc" "C14663"
+			(at 173.99 33.02 0)
+			(effects
+				(font
+					(size 1.27 1.27)
+				)
+				(hide yes)
+			)
+		)
 		(pin "1"
 		)
@@
 			)
 		)
-		(property "Value" "1A, 30V"
+		(property "Value" "2A, 30V"
 			(at 58.166 122.428 0)
 			(effects
@@
 			)
 		)
-		(property "MPN" "DFLS130-7"
+		(property "MPN" "DFLS230LH-7"
 			(at 59.69 124.46 0)
 			(effects
@@
 			)
 		)
-		(property "jlc" "C150474"
+		(property "jlc" "C2960361"
 			(at 59.69 124.46 0)
 			(effects
@@
 			)
 		)
+		(property "jlc" "C14663"
+			(at 224.79 29.21 0)
+			(effects
+				(font
+					(size 1.27 1.27)
+				)
+				(hide yes)
+			)
+		)
 		(pin "1"
 		)
@@
 			)
 		)
+		(property "jlc" "C14663"
+			(at 168.91 54.61 0)
+			(effects
+				(font
+					(size 1.27 1.27)
+				)
+				(hide yes)
+			)
+		)
 		(pin "1"
 		)
@@
 			)
 		)
+		(property "jlc" "C14663"
+			(at 76.2 162.56 0)
+			(effects
+				(font
+					(size 1.27 1.27)
+				)
+				(hide yes)
+			)
+		)
 		(pin "1"
 		)
@@
 			)
 		)
+		(property "jlc" "C2286"
+			(at 227.33 149.86 0)
+			(effects
+				(font
+					(size 1.27 1.27)
+				)
+				(hide yes)
+			)
+		)
 		(pin "1"
 		)
@@
 			)
 		)
+		(property "jlc" "C14663"
+			(at 167.64 33.02 0)
+			(effects
+				(font
+					(size 1.27 1.27)
+				)
+				(hide yes)
+			)
+		)
 		(pin "1"
 		)
@@
 			)
 		)
+		(property "jlc" "C14663"
+			(at 147.32 33.02 0)
+			(effects
+				(font
+					(size 1.27 1.27)
+				)
+				(hide yes)
+			)
+		)
 		(pin "1"
 		)
@@
 			)
 		)
+		(property "jlc" "C15849"
+			(at 176.53 54.61 0)
+			(effects
+				(font
+					(size 1.27 1.27)
+				)
+				(hide yes)
+			)
+		)
 		(pin "1"
 		)
@@
 			)
 		)
+		(property "jlc" "C14663"
+			(at 80.01 57.15 0)
+			(effects
+				(font
+					(size 1.27 1.27)
+				)
+				(hide yes)
+			)
+		)
 		(pin "1"
 		)
@@
 			)
 		)
+		(property "jlc" "C49257"
+			(at 129.54 151.13 0)
+			(effects
+				(font
+					(size 1.27 1.27)
+				)
+				(hide yes)
+			)
+		)
 		(pin "3"
 		)
@@
 			)
 		)
+		(property "jlc" "C14663"
+			(at 160.02 33.02 0)
+			(effects
+				(font
+					(size 1.27 1.27)
+				)
+				(hide yes)
+			)
+		)
 		(pin "1"
 		)
@@
 			)
 		)
+		(property "jlc" "C15849"
+			(at 203.2 53.34 0)
+			(effects
+				(font
+					(size 1.27 1.27)
+				)
+				(hide yes)
+			)
+		)
 		(pin "1"
 		)
@@
 			)
 		)
+		(property "jlc" "C14663"
+			(at 180.34 33.02 0)
+			(effects
+				(font
+					(size 1.27 1.27)
+				)
+				(hide yes)
+			)
+		)
 		(pin "1"
 		)
@@
 			(at 162.56 54.61 0)
 			(effects
+				(font
+					(size 1.27 1.27)
+				)
+				(hide yes)
+			)
+		)
+		(property "jlc" "C14663"
+			(at 162.56 54.61 0)
+			(effects

Commit message: jlc codes filled
Parts:
- R1, R7: jlc (none) -> C25804
- R10, R3, R4: jlc (none) -> C23186
- R2, R8: jlc (none) -> C21190
- R27, R28, R29, R30: jlc (none) -> C22775
- R5, R6: jlc (none) -> C25190
- U5: jlc (none) -> C2040
- U7: jlc (none) -> C131025
Changed lines of the file:
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@@
 			)
 		)
+		(property "jlc" "C25190"
+			(at 78.74 139.7 0)
+			(effects
+				(font
+					(size 1.27 1.27)
+				)
+				(hide yes)
+			)
+		)
 		(pin "1"
 		)
@@
 			)
 		)
+		(property "jlc" "C21190"
+			(at 40.64 38.1 0)
+			(effects
+				(font
+					(size 1.27 1.27)
+				)
+				(hide yes)
+			)
+		)
 		(pin "1"
 		)
@@
 			)
 		)
+		(property "jlc" "C23186"
+			(at 227.33 142.24 0)
+			(effects
+				(font
+					(size 1.27 1.27)
+				)
+				(hide yes)
+			)
+		)
 		(pin "1"
 		)
@@
 			)
 		)
+		(property "jlc" "C25190"
+			(at 78.74 142.24 0)
+			(effects
+				(font
+					(size 1.27 1.27)
+				)
+				(hide yes)
+			)
+		)
 		(pin "1"
 		)
@@
 			)
 		)
+		(property "jlc" "C21190"
+			(at 152.4 127 0)
+			(effects
+				(font
+					(size 1.27 1.27)
+				)
+				(hide yes)
+			)
+		)
 		(pin "1"
 		)
@@
 			)
 		)
+		(property "jlc" "C23186"
+			(at 58.42 132.08 0)
+			(effects
+				(font
+					(size 1.27 1.27)
+				)
+				(hide yes)
+			)
+		)
 		(pin "1"
 		)
@@
 			)
 		)
+		(property "jlc" "C25804"
+			(at 151.13 63.5 0)
+			(effects
+				(font
+					(size 1.27 1.27)
+				)
+				(hide yes)
+			)
+		)
 		(pin "1"
 		)
@@
 			)
 		)
+		(property "jlc" "C22775"
+			(at 219.71 74.93 0)
+			(effects
+				(font
+					(size 1.27 1.27)
+				)
+				(hide yes)
+			)
+		)
 		(pin "1"
 		)
@@
 			)
 		)
+		(property "jlc" "C22775"
+			(at 219.71 72.39 0)
+			(effects
+				(font
+					(size 1.27 1.27)
+				)
+				(hide yes)
+			)
+		)
 		(pin "1"
 		)
@@
 			)
 		)
+		(property "jlc" "C25804"
+			(at 50.8 38.1 0)
+			(effects
+				(font
+					(size 1.27 1.27)
+				)
+				(hide yes)
+			)
+		)
 		(pin "1"
 		)
@@
 			)
 		)
+		(property "jlc" "C131025"
+			(at 64.77 58.42 0)
+			(effects
+				(font
+					(size 1.27 1.27)
+				)
+				(hide yes)
+			)
+		)
 		(pin "1"
 		)
@@
 			)
 		)
+		(property "jlc" "C23186"
+			(at 58.42 129.54 0)
+			(effects
+				(font
+					(size 1.27 1.27)
+				)
+				(hide yes)
+			)
+		)
 		(pin "1"
 		)
@@
 			)
 		)
+		(property "jlc" "C22775"
+			(at 266.7 71.12 0)
+			(effects
+				(font
+					(size 1.27 1.27)
+				)
+				(hide yes)
+			)
+		)
 		(pin "1"
 		)
@@
 			)
 		)
+		(property "jlc" "C2040"
+			(at 187.96 105.41 0)
+			(effects
+				(font
+					(size 1.27 1.27)
+				)
+				(hide yes)
+			)
+		)
 		(pin "16"
 		)
@@
 			(at 266.7 86.36 0)
 			(effects
+				(font
+					(size 1.27 1.27)
+				)
+				(hide yes)
+			)
+		)
+		(property "jlc" "C22775"
+			(at 266.7 86.36 0)
+			(effects

Commit message: routing in progress
Parts:
- added R57: 1Meg 1%, Resistor_SMD:R_0603_1608Metric_Pad0.98x0.95mm_HandSolder, symbol Device:R_Small
- R7: now left out of the parts list
Connections:
- net at C17.1, R8.2, Y1.1: now also R57.2
- net at C18.1, U5.20 (XIN), Y1.3: now also R57.1
Other:
- moved on the sheet: C17, C18
Changed lines of the file:
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@@
 	)
 	(junction
+		(at 133.35 109.22)
+		(diameter 0)
+		(color 0 0 0 0)
+	)
+	(junction
 		(at 151.13 67.31)
 		(diameter 0)
@@
 	)
 	(junction
+		(at 133.35 127)
+		(diameter 0)
+		(color 0 0 0 0)
+	)
+	(junction
 		(at 80.01 73.66)
 		(diameter 0)
@@
 	(wire
 		(pts
-			(xy 139.7 109.22) (xy 146.05 109.22)
+			(xy 128.27 109.22) (xy 133.35 109.22)
 		)
 		(stroke
@@
 	(wire
 		(pts
+			(xy 133.35 109.22) (xy 133.35 115.57)
+		)
+		(stroke
+			(width 0)
+			(type default)
+		)
+	)
+	(wire
+		(pts
 			(xy 60.96 129.54) (xy 68.58 129.54)
 		)
@@
 	(wire
 		(pts
+			(xy 133.35 120.65) (xy 133.35 127)
+		)
+		(stroke
+			(width 0)
+			(type default)
+		)
+	)
+	(wire
+		(pts
 			(xy 52.07 132.08) (xy 55.88 132.08)
 		)
@@
 	(wire
 		(pts
+			(xy 133.35 109.22) (xy 146.05 109.22)
+		)
+		(stroke
+			(width 0)
+			(type default)
+		)
+	)
+	(wire
+		(pts
 			(xy 154.94 127) (xy 160.02 127)
 		)
@@
 	(wire
 		(pts
+			(xy 133.35 127) (xy 128.27 127)
+		)
+		(stroke
+			(width 0)
+			(type default)
+		)
+	)
+	(wire
+		(pts
 			(xy 256.54 71.12) (xy 261.62 71.12)
 		)
@@
 	(wire
 		(pts
-			(xy 146.05 127) (xy 139.7 127)
+			(xy 146.05 127) (xy 133.35 127)
 		)
 		(stroke
@@
 	(symbol
 		(lib_id "power:GND")
-		(at 134.62 109.22 270)
+		(at 123.19 109.22 270)
 		(unit 1)
 		(exclude_from_sim no)
@@
 		(dnp no)
 		(property "Reference" "#PWR061"
-			(at 128.27 109.22 0)
+			(at 116.84 109.22 0)
 			(effects
 				(font
@@
 		)
 		(property "Value" "GND"
-			(at 131.064 109.22 0)
+			(at 119.634 109.22 0)
 			(effects
 				(font
@@
 		)
 		(property "Footprint" ""
-			(at 134.62 109.22 0)
+			(at 123.19 109.22 0)
 			(effects
 				(font
@@
 		)
 		(property "Datasheet" ""
-			(at 134.62 109.22 0)
+			(at 123.19 109.22 0)
 			(effects
 				(font
@@
 		)
 		(property "Description" "Power symbol creates a global label with name \"GND\" , ground"
-			(at 134.62 109.22 0)
+			(at 123.19 109.22 0)
 			(effects
 				(font
@@
 		)
 		(property "Value" "GND"
-			(at 137.414 118.11 0)
+			(at 137.414 118.364 0)
 			(effects
 				(font
@@
 		(unit 1)
 		(exclude_from_sim no)
-		(in_bom yes)
+		(in_bom no)
 		(on_board yes)
 		(dnp yes)
@@
 	(symbol
 		(lib_id "Device:C_Small")
-		(at 137.16 127 270)
+		(at 125.73 127 270)
 		(unit 1)
 		(exclude_from_sim no)
@@
 		(dnp no)
 		(property "Reference" "C17"
-			(at 138.176 125.73 90)
+			(at 126.746 125.73 90)
 			(effects
 				(font
@@
 		)
 		(property "Value" "22p 50V"
-			(at 132.08 129.54 90)
+			(at 120.65 129.54 90)
 			(effects
 				(font
@@
 		)
 		(property "Footprint" "Capacitor_SMD:C_0603_1608Metric_Pad1.08x0.95mm_HandSolder"
-			(at 137.16 127 0)
+			(at 125.73 127 0)
 			(effects
 				(font
@@
 		)
 		(property "Datasheet" "~"
-			(at 137.16 127 0)
+			(at 125.73 127 0)
 			(effects
 				(font
@@
 		)
 		(property "Description" ""
-			(at 137.16 127 0)
+			(at 125.73 127 0)
 			(effects
 				(font
@@
 		)
 		(property "jlc" "C1653"
-			(at 137.16 127 90)
+			(at 125.73 127 90)
 			(effects
 				(font
@@
 	)
 	(symbol
+		(lib_id "Device:R_Small")
+		(at 133.35 118.11 0)
+		(unit 1)
+		(exclude_from_sim no)
+		(in_bom no)
+		(on_board yes)
+		(dnp yes)
+		(property "Reference" "R57"
+			(at 127 117.094 0)
+			(effects
+				(font
+					(size 1.27 1.27)
+				)
+				(justify left)
+			)
+		)
+		(property "Value" "1Meg 1%"
+			(at 123.444 118.872 0)
+			(effects
+				(font
+					(size 1.27 1.27)
+				)
+				(justify left)
+			)
+		)
+		(property "Footprint" "Resistor_SMD:R_0603_1608Metric_Pad0.98x0.95mm_HandSolder"
+			(at 133.35 118.11 0)
+			(effects
+				(font
+					(size 1.27 1.27)
+				)
+				(hide yes)
+			)
+		)
+		(property "Datasheet" "~"
+			(at 133.35 118.11 0)
+			(effects
+				(font
+					(size 1.27 1.27)
+				)
+				(hide yes)
+			)
+		)
+		(property "Description" ""
+			(at 133.35 118.11 0)
+			(effects
+				(font
+					(size 1.27 1.27)
+				)
+				(hide yes)
+			)
+		)
+		(property "jlc" ""
+			(at 133.35 118.11 0)
+			(effects
+				(font
+					(size 1.27 1.27)
+				)
+				(hide yes)
+			)
+		)
+		(pin "1"
+		)
+		(pin "2"
+		)
+		(instances
+			(project "beam_kit_1"
+				(path "/3a707576-1044-44db-8cf8-deb84fe605c8/35bb5101-2bc6-4b84-84b4-e3f71c5fc9a9"
+					(reference "R57")
+					(unit 1)
+				)
+			)
+		)
+	)
+	(symbol
 		(lib_id "Connector_Generic:Conn_01x03")
 		(at 129.54 151.13 180)
@@
 	(symbol
 		(lib_id "Device:C_Small")
-		(at 137.16 109.22 270)
+		(at 125.73 109.22 270)
 		(unit 1)
 		(exclude_from_sim no)
@@
 		(dnp no)
 		(property "Reference" "C18"
-			(at 138.176 107.95 90)
+			(at 126.746 107.95 90)
 			(effects
 				(font
@@
 		)
 		(property "Value" "22p 50V"
-			(at 132.08 111.76 90)
+			(at 120.65 111.76 90)
 			(effects
 				(font
@@
 		)
 		(property "Footprint" "Capacitor_SMD:C_0603_1608Metric_Pad1.08x0.95mm_HandSolder"
-			(at 137.16 109.22 0)
+			(at 125.73 109.22 0)
 			(effects
 				(font
@@
 		)
 		(property "Datasheet" "~"
-			(at 137.16 109.22 0)
+			(at 125.73 109.22 0)
 			(effects
 				(font
@@
 		)
 		(property "Description" ""
-			(at 137.16 109.22 0)
+			(at 125.73 109.22 0)
 			(effects
 				(font
@@
 		)
 		(property "jlc" "C1653"
-			(at 137.16 109.22 90)
+			(at 125.73 109.22 90)
 			(effects
 				(font
@@
 	(symbol
 		(lib_id "power:GND")
-		(at 134.62 127 270)
+		(at 123.19 127 270)
 		(unit 1)
 		(exclude_from_sim no)
@@
 		(dnp no)
 		(property "Reference" "#PWR062"
-			(at 128.27 127 0)
+			(at 116.84 127 0)
 			(effects
 				(font
@@
 		)
 		(property "Value" "GND"
-			(at 131.064 127 0)
+			(at 119.634 127 0)
 			(effects
 				(font
@@
 		)
 		(property "Footprint" ""
-			(at 134.62 127 0)
+			(at 123.19 127 0)
 			(effects
 				(font
@@
 		)
 		(property "Datasheet" ""
-			(at 134.62 127 0)
+			(at 123.19 127 0)
 			(effects
 				(font
@@
 		)
 		(property "Description" "Power symbol creates a global label with name \"GND\" , ground"
-			(at 134.62 127 0)
+			(at 123.19 127 0)
 			(effects
 				(font

Commit message: layout done
Parts:
- added C73: 100u 6V3 Tantal, Capacitor_Tantalum_SMD:CP_EIA-3528-21_Kemet-B_Pad1.50x2.35mm_HandSolder, symbol Device:C_Polarized_Small
Connections:
- net +3.3V: now also C73.1
- net GND: now also C73.2
Changed lines of the file:
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@@
 	)
 	(symbol
+		(lib_id "power:GND")
+		(at 130.81 31.75 0)
+		(unit 1)
+		(exclude_from_sim no)
+		(in_bom yes)
+		(on_board yes)
+		(dnp no)
+		(fields_autoplaced yes)
+		(property "Reference" "#PWR0208"
+			(at 130.81 38.1 0)
+			(effects
+				(font
+					(size 1.27 1.27)
+				)
+				(hide yes)
+			)
+		)
+		(property "Value" "GND"
+			(at 130.81 36.83 0)
+			(effects
+				(font
+					(size 1.27 1.27)
+				)
+			)
+		)
+		(property "Footprint" ""
+			(at 130.81 31.75 0)
+			(effects
+				(font
+					(size 1.27 1.27)
+				)
+				(hide yes)
+			)
+		)
+		(property "Datasheet" ""
+			(at 130.81 31.75 0)
+			(effects
+				(font
+					(size 1.27 1.27)
+				)
+				(hide yes)
+			)
+		)
+		(property "Description" "Power symbol creates a global label with name \"GND\" , ground"
+			(at 130.81 31.75 0)
+			(effects
+				(font
+					(size 1.27 1.27)
+				)
+				(hide yes)
+			)
+		)
+		(pin "1"
+		)
+		(instances
+			(project "beam_kit_1"
+				(path "/3a707576-1044-44db-8cf8-deb84fe605c8/35bb5101-2bc6-4b84-84b4-e3f71c5fc9a9"
+					(reference "#PWR0208")
+					(unit 1)
+				)
+			)
+		)
+	)
+	(symbol
 		(lib_id "power:+3.3V")
 		(at 213.36 33.02 0)
@@
 	)
 	(symbol
+		(lib_id "Device:C_Polarized_Small")
+		(at 130.81 29.21 0)
+		(mirror y)
+		(unit 1)
+		(exclude_from_sim no)
+		(in_bom yes)
+		(on_board yes)
+		(dnp no)
+		(property "Reference" "C73"
+			(at 128.27 27.3938 0)
+			(effects
+				(font
+					(size 1.27 1.27)
+				)
+				(justify left)
+			)
+		)
+		(property "Value" "100u 6V3 Tantal"
+			(at 128.27 29.9338 0)
+			(effects
+				(font
+					(size 1.27 1.27)
+				)
+				(justify left)
+			)
+		)
+		(property "Footprint" "Capacitor_Tantalum_SMD:CP_EIA-3528-21_Kemet-B_Pad1.50x2.35mm_HandSolder"
+			(at 130.81 29.21 0)
+			(effects
+				(font
+					(size 1.27 1.27)
+				)
+				(hide yes)
+			)
+		)
+		(property "Datasheet" "~"
+			(at 130.81 29.21 0)
+			(effects
+				(font
+					(size 1.27 1.27)
+				)
+				(hide yes)
+			)
+		)
+		(property "Description" "Polarized capacitor, small symbol"
+			(at 130.81 29.21 0)
+			(effects
+				(font
+					(size 1.27 1.27)
+				)
+				(hide yes)
+			)
+		)
+		(property "jlc" "C16133"
+			(at 130.81 29.21 0)
+			(effects
+				(font
+					(size 1.27 1.27)
+				)
+				(hide yes)
+			)
+		)
+		(pin "1"
+		)
+		(pin "2"
+		)
+		(instances
+			(project "beam_kit_1"
+				(path "/3a707576-1044-44db-8cf8-deb84fe605c8/35bb5101-2bc6-4b84-84b4-e3f71c5fc9a9"
+					(reference "C73")
+					(unit 1)
+				)
+			)
+		)
+	)
+	(symbol
 		(lib_id "power:GND")
 		(at 160.02 35.56 0)
@@
 					(unit 1)
 				)
+			)
+		)
+	)
+	(symbol
+		(lib_id "power:+3.3V")
+		(at 130.81 26.67 0)
+		(unit 1)
+		(exclude_from_sim no)
+		(in_bom yes)
+		(on_board yes)
+		(dnp no)
+		(property "Reference" "#PWR0237"
+			(at 130.81 30.48 0)
+			(effects
+				(font
+					(size 1.27 1.27)
+				)
+				(hide yes)
+			)
+		)
+		(property "Value" "+3.3V"
+			(at 129.794 22.606 0)
+			(effects
+				(font
+					(size 1.27 1.27)
+				)
+			)
+		)
+		(property "Footprint" ""
+			(at 130.81 26.67 0)
+			(effects
+				(font
+					(size 1.27 1.27)
+				)
+				(hide yes)
+			)
+		)
+		(property "Datasheet" ""
+			(at 130.81 26.67 0)
+			(effects
+				(font
+					(size 1.27 1.27)
+				)
+				(hide yes)
+			)
+		)
+		(property "Description" "Power symbol creates a global label with name \"+3.3V\""
+			(at 130.81 26.67 0)
+			(effects
+				(font
+					(size 1.27 1.27)
+				)
+				(hide yes)
+			)
+		)
+		(pin "1"
+		)
+		(instances
+			(project "beam_kit_1"
+				(path "/3a707576-1044-44db-8cf8-deb84fe605c8/35bb5101-2bc6-4b84-84b4-e3f71c5fc9a9"
+					(reference "#PWR0237")
+					(unit 1)
+				)

Commit message: final version
Parts:
- C10, C11, C12, C13, C15, C16, C20, C4, C6, C7, C8, C9: JLC (none) -> C14663
- C14, C5: JLC (none) -> C15849
- C17, C18: JLC (none) -> C1653
- C73: JLC (none) -> C16133
- D1: JLC (none) -> C495220
- D2: JLC (none) -> C2960361
- D3: JLC (none) -> C2286
- J3: JLC (none) -> C134092; jlc 1054500101 -> C134092
- J4: JLC (none) -> C49257
- R1, R7: JLC (none) -> C25804
- R10, R3, R4: JLC (none) -> C23186
- R2, R8: JLC (none) -> C21190
- R27, R28, R29, R30: JLC (none) -> C22775
- R5, R6: JLC (none) -> C25190
- SW1, SW2: JLC (none) -> C231329
- U5: JLC (none) -> C2040
- U7: JLC (none) -> C131025
- Y1: JLC (none) -> C9002
